File: schematics/controller.sch (KiCad schematic (older format))
At the start: 29 parts, among them J1 JACK STEREO, SW1 MOMENTARY, SW10 MOMENTARY, SW2 MOMENTARY, SW3 MOMENTARY, SW4 MOMENTARY, SW5 MOMENTARY, SW6 MOMENTARY, SW7 MOMENTARY, SW8 MOMENTARY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

Commit message: Update controller schematics
Connections:
- net ICSP-3 is gone; now on net RV6W: DP1.~ (W6)
- net ICSP-4 is gone; now on net RV6W: DP1.~ (W6)
- new net: A1.~ (RESET), DP1.~ (W6)
- new net 51: DP1.~ (W6)
- new net 52: DP1.~ (W6)
Changed lines of the file:
@@
 Sheet 1 1
 Title "PREAMPino control unit"
-Date "1 may 2016"
+Date "13 may 2016"
 Rev "1"
 Comp ""
@@
 ValveCaster\nVolume
 Text GLabel 19000 2850 0    60   Input ~ 0
-ICSP-4
+51
 Text GLabel 19650 2950 0    60   Input ~ 0
-ICSP-3
+52
 Text Notes 14250 6500 0    60   ~ 0
 Down\n
